Commit message: update

File: ros2_ws/src/balancing-robot-description/urdf/robot.urdf (robot description, URDF)
Before this commit: robot balancing_robot, 1 links, 0 joints
Links:
- added link left_wheel, mass 0.2; collision cylinder length=0.04 radius=0.05; visual cylinder length=0.04 radius=0.05
- added link right_wheel, mass 0.2; collision cylinder length=0.04 radius=0.05; visual cylinder length=0.04 radius=0.05
- link base_link: mass None -> 1.0; geometry collision box size=0.2 0.3 0.1; visual box size=0.2 0.3 0.1
Joints:
- added joint left_wheel_joint: type continuous, parent base_link, child left_wheel, origin xyz=0 0.17 0 rpy=-1.5708 0 0, axis 0 0 1
- added joint right_wheel_joint: type continuous, parent base_link, child right_wheel, origin xyz=0 -0.17 0 rpy=-1.5708 0 0, axis 0 0 1

Commit message: Add Controller node for calculating PID output for robot, fix imu not transferring data to controller node

File: ros2_ws/src/balancing-robot-description/urdf/robot.urdf (robot description, URDF)
Before this commit: robot balancing_robot, 3 links, 2 joints
Links:
- added link base_footprint
- link base_link: mass 1.0 -> 0.89; geometry collision box size=0.08 0.19 0.12; visual box size=0.08 0.19 0.12
- link left_wheel: geometry collision cylinder length=0.04 radius=0.04; visual cylinder length=0.04 radius=0.04
- link right_wheel: geometry collision cylinder length=0.04 radius=0.04; visual cylinder length=0.04 radius=0.04
Joints:
- added joint base_footprint_joint: type fixed, parent base_footprint, child base_link, origin xyz=0 0 0 rpy=0 0 0
- joint left_wheel_joint: origin xyz=0 0.17 0 rpy=-1.5708 0 0 -> xyz=0 0.14 0 rpy=-1.5708 0 0
- joint right_wheel_joint: origin xyz=0 -0.17 0 rpy=-1.5708 0 0 -> xyz=0 -0.14 0 rpy=-1.5708 0 0

Commit message: add gyroscope y measurement to fuse with accelerometer measurement for correction, add API for getting P I D values for logging

File: ros2_ws/src/balancing-robot-description/urdf/robot.urdf (robot description, URDF)
Before this commit: robot balancing_robot, 4 links, 3 joints
Links:
- link base_footprint: mass None -> 0.001
Joints:
- joint base_footprint_joint: origin xyz=0 0 0 rpy=0 0 0 -> xyz=0 0 0 rpy=0 0.035 0

Commit message: Reconfigure PID class so that ouput is in range -1 to 1, output will be percentage Reconfigure urdf file so that it is more stable, like real hardware Change from using velocity to control motor to using torque, create new config file Todo: reconfigure control class to talk to new control topic, setup.

File: ros2_ws/src/balancing-robot-description/urdf/robot.urdf (robot description, URDF)
Before this commit: robot balancing_robot, 4 links, 3 joints
Links:
- added link top_plate, mass 0.4; collision box size=0.065 0.14 0.005; visual box size=0.065 0.14 0.005
- link base_footprint: mass 0.001 -> None
- link base_link: mass 0.89 -> 0.5; geometry collision box size=0.065 0.14 0.005; visual box size=0.065 0.14 0.005
- link left_wheel: mass 0.2 -> 0.1; geometry collision cylinder length=0.025 radius=0.0325; visual cylinder length=0.025 radius=0.0325
- link right_wheel: mass 0.2 -> 0.1; geometry collision cylinder length=0.025 radius=0.0325; visual cylinder length=0.025 radius=0.0325
Joints:
- removed joint base_footprint_joint
- added joint base_joint: type fixed, parent base_footprint, child base_link, origin xyz=0 0 0.0325 rpy=0 0.035 0
- added joint spacer_joint: type fixed, parent base_link, child top_plate, origin xyz=0 0 0.085 rpy=0 0 0
- joint left_wheel_joint: limit (none) -> effort=0.49 velocity=34.8; origin xyz=0 0.14 0 rpy=-1.5708 0 0 -> xyz=0 0.08 0 rpy=-1.5708 0 0
- joint right_wheel_joint: limit (none) -> effort=0.49 velocity=34.8; origin xyz=0 -0.14 0 rpy=-1.5708 0 0 -> xyz=0 -0.08 0 rpy=-1.5708 0 0
